File: guy.kicad_pcb (KiCad board)
At the start: 2 copper layers, 17 parts, among them J2 Barrel_Jack_MountingPin, J3 Conn_Coaxial, Q1 2N3906, SW1 SW_Wuerth_450301014042, SW2 SW_Nidec_CAS-120A1, Y2 Crystal

Commit message: Add files via upload
Parts:
- removed SW2: SW_Nidec_CAS-120A1, Button_Switch_SMD:Nidec_Copal_CAS-120A
- added J1: AudioJack2_SwitchT, Connector_Audio:Jack_3.5mm_Lumberg_1503_07_Horizontal, F.Cu at (170.2, 51.5)
- moved C3 20.3 mm to (150.0, 72.5), turned to 180 degrees
Routing:
- net Net-(C1-Pad2): track 75.2 -> 104.7 mm
- net (no net): track 5.65 -> 0.00 mm
- net Net-(Q1-E): track 32.4 -> 36.9 mm
Other:
- board outline added: 70.5 x 51 mm
- board text added: "2024"
- board text added: "BrokeCW"
- board text added: "HackClub"
- board text added: "Rose Weatherly"
