File: BrokeCW1.kicad_pcb (KiCad board)
At the start: 2 copper layers, 44 parts, among them J1 Barrel_Jack_MountingPin, J10 AudioJack3_Radio, J2 Conn_Coaxial, J3 AudioJack3_Ground, J4 AudioJack3_Ground, J6 Conn_01x03_Pin, J7 Conn_01x15_PinLeft, J8 Conn_01x15_PinRight, J9 AudioJack3_Key, Q1 9013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

Commit message: Add files via upload
Parts:
- removed R5, R7: R10K, Resistor_SMD:R_1210_3225Metric
- removed SW2, SW3, SW4, SW5, SW6: CK_KMS2xxGP, Button_Switch_SMD:SW_SPST_CK_KMS2xxGP
- added J5: Conn_01x03_Pin, Connector_Hirose:Hirose_DF13-03P-1.25DSA_1x03_P1.25mm_Vertical, F.Cu at (157.5, 59.0)
- added SW7: SW_Coded_SH-7050, Button_Switch_SMD:Nidec_Copal_SH-7010B, F.Cu at (63.5, 74.0)
- C1, C2: footprint Capacitor_SMD:C_0805_2012Metric -> Capacitor_SMD:C_0603_1608Metric
- C3, C4: value C0.1uF -> C
- C5, C6: footprint Capacitor_SMD:C_0201_0603Metric -> Capacitor_SMD:C_0805_2012Metric
- C7: footprint Capacitor_THT:C_Disc_D5.1mm_W3.2mm_P5.00mm -> Capacitor_SMD:C_0805_2012Metric
- C8, C9: footprint Capacitor_SMD:C_0402_1005Metric -> Capacitor_SMD:C_0805_2012Metric
- D1: footprint Diode_THT:D_DO-41_SOD81_P7.62mm_Horizontal -> Diode_SMD:D_SOD-323
- D2, D3: footprint LED_SMD:LED_0402_1005Metric -> LED_SMD:LED_0805_2012Metric
- Q1, Q2: footprint Package_TO_SOT_THT:TO-92_Inline -> Package_TO_SOT_SMD:SOT-23
- R1: footprint Resistor_SMD:R_2512_6332Metric -> Resistor_SMD:R_0805_2012Metric
- R2: footprint Resistor_SMD:R_1210_3225Metric -> Resistor_SMD:R_0603_1608Metric
- R3: footprint Resistor_SMD:R_1210_3225Metric -> Resistor_SMD:R_1206_3216Metric
- R4: footprint Resistor_SMD:R_2512_6332Metric -> Resistor_SMD:R_1206_3216Metric
- R6: footprint Resistor_THT:R_Axial_DIN0414_L11.9mm_D4.5mm_P15.24mm_Horizontal -> Resistor_SMD:R_1206_3216Metric
- R8: value R_Small -> R; footprint Resistor_SMD:R_0201_0603Metric -> Resistor_SMD:R_0603_1608Metric
- moved J9 108.1 mm to (50.8, 52.9)
- moved RV3 106.9 mm to (47.0, 69.5)
- moved J8 106.8 mm to (101.5, 51.5)
- moved D3 106.7 mm to (113.0, 60.0)
- moved J10 106.6 mm to (119.2, 76.0)
- moved J7 105.8 mm to (85.5, 51.5)
- moved R8 104.5 mm to (119.3, 56.5)
- moved C9 88.8 mm to (216.9, 41.9), turned to 180 degrees
- moved L2 82.5 mm to (216.0, 47.9)
- moved C8 80.6 mm to (207.4, 46.4), turned to 90 degrees
- moved SW1 72.2 mm to (144.0, 48.7)
- moved J1 63.8 mm to (137.9, 43.1), turned to -90 degrees
- moved C7 62.0 mm to (196.4, 46.4), turned to 180 degrees
- moved D2 51.8 mm to (188.0, 65.5), turned to 180 degrees
- moved RV2 49.6 mm to (176.0, 94.5), turned to 90 degrees
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Connections:
- C5 pad 2: Net-(D2-A) -> Net-(D1-A)
- C6 pad 2: Net-(D1-A) -> Net-(D2-A)
- J7 pad 10: unconnected-(J7-Pin_10-Pad10) -> Net-(J7-Pin_10)
- J7 pad 12: unconnected-(J7-Pin_12-Pad12) -> Net-(J7-Pin_12)
- J7 pad 4: unconnected-(J7-Pin_4-Pad4) -> Net-(J7-Pin_4)
- J7 pad 5: unconnected-(J7-Pin_5-Pad5) -> Net-(J7-Pin_5)
- J8 pad 6: Net-(J8-Pin_6) -> unconnected-(J8-Pin_6-Pad6)
- J9 pad T: Net-(J9-PadG) -> Net-(J7-Pin_12)
- RV3 pad 1: unconnected-(RV3-Pad1) -> Net-(J7-Pin_10)
- RV3 pad 2: unconnected-(RV3-Pad2) -> Net-(J7-Pin_5)
- RV3 pad 3: Net-(J9-PadG) -> Net-(J7-Pin_12)
Routing:
- net Net-(D2-K): track 0.00 -> 265.0 mm
- net Net-(D1-A): track 0.00 -> 231.0 mm
- net Net-(D2-A): track 0.00 -> 115.1 mm
- net Net-(J7-Pin_12): track 0.00 -> 54.3 mm
- net Net-(Q2-C): track 0.00 -> 51.7 mm
- net Net-(J5-Pin_1): track 0.00 -> 27.1 mm
- net Net-(R6-Pad2): track 0.00 -> 26.1 mm
- net Net-(J7-Pin_8): track 0.00 -> 25.9 mm
- net Net-(U1-+): track 0.00 -> 22.5 mm
- net Net-(J7-Pin_10): track 0.00 -> 19.2 mm
- net Net-(C7-Pad1): track 0.00 -> 17.6 mm
- net Net-(J2-In): track 0.00 -> 16.1 mm
- net Net-(C2-Pad2): track 0.00 -> 14.1 mm
- net Net-(J8-Pin_12): track 0.00 -> 13.8 mm
- net Net-(J8-Pin_9): track 0.00 -> 12.9 mm
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Other:
- board outline added: 222.2 x 72.2 mm
