File: BrokeCW.kicad_sch (KiCad schematic)
At the start: 45 parts, among them J1 Barrel_Jack_MountingPin, J10 AudioJack3_Radio, J2 Conn_Coaxial, J3 AudioJack3_Ground, J4 AudioJack3_Ground, J5 Conn_01x03_Pin, J6 Conn_01x03_Pin, J7 Conn_01x15_PinLeft, J8 Conn_01x15_PinRight, J9 AudioJack3_Key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

Commit message: Add files via upload
Parts:
- C3, C4: value C0.1uF -> C; footprint Capacitor_SMD:C_0603_1608Metric -> Capacitor_THT:C_Disc_D5.1mm_W3.2mm_P5.00mm
- C5, C6: footprint Capacitor_SMD:C_0201_0603Metric -> Capacitor_THT:C_Disc_D7.0mm_W2.5mm_P5.00mm
Connections:
- net at C3.2, C8.2, C9.2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: now also C5.2; no longer C6.2
- net at D2.2 (A), L1.1, L3.1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: now also C6.2; no longer C5.2
- net at J7.12 (Pin_12): now also J9.G, J9.T, RV3.3, SW2.1, SW3.1, SW4.1, SW5.1, SW6.1
- net at J7.4 (Pin_4): now also R5.1, SW3.2
- net at J7.5 (Pin_5): now also RV3.2
- net at J7.8 (Pin_8), R7.1, SW4.2: no longer RV3.3

Commit message: Add files via upload
Parts:
- J5: footprint (none) -> Connector_Hirose:Hirose_DF13-03P-1.25DSA_1x03_P1.25mm_Vertical
Connections:
- net at C5.1, C6.1, Q1.3 (B)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: now also J5.1 (Pin_1), J5.2 (Pin_2), J5.3 (Pin_3)
Changed lines of the file:
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@@
 	)
 	(junction
+		(at 130.81 43.18)
+		(diameter 0)
+		(color 0 0 0 0)
+	)
+	(junction
 		(at 182.88 82.55)
 		(diameter 0)
@@
 	)
 	(junction
+		(at 133.35 43.18)
+		(diameter 0)
+		(color 0 0 0 0)
+	)
+	(junction
 		(at 41.91 152.4)
 		(diameter 0)
@@
 	)
 	(junction
+		(at 128.27 43.18)
+		(diameter 0)
+		(color 0 0 0 0)
+	)
+	(junction
 		(at 58.42 170.18)
 		(diameter 0)
@@
 	(wire
 		(pts
+			(xy 133.35 43.18) (xy 146.05 43.18)
+		)
+		(stroke
+			(width 0)
+			(type default)
+		)
+	)
+	(wire
+		(pts
 			(xy 133.35 30.48) (xy 146.05 30.48)
 		)
@@
 	(wire
 		(pts
-			(xy 128.27 43.18) (xy 146.05 43.18)
+			(xy 128.27 43.18) (xy 130.81 43.18)
 		)
 		(stroke
@@
 	(wire
 		(pts
+			(xy 128.27 38.1) (xy 128.27 43.18)
+		)
+		(stroke
+			(width 0)
+			(type default)
+		)
+	)
+	(wire
+		(pts
 			(xy 262.89 80.01) (xy 262.89 101.6)
 		)
@@
 	(wire
 		(pts
+			(xy 130.81 43.18) (xy 133.35 43.18)
+		)
+		(stroke
+			(width 0)
+			(type default)
+		)
+	)
+	(wire
+		(pts
 			(xy 160.02 114.3) (xy 176.53 114.3)
 		)
@@
 	)
 	(symbol
-		(lib_id "Connector:Conn_01x03_Pin")
-		(at 130.81 43.18 270)
-		(unit 1)
-		(exclude_from_sim no)
-		(in_bom yes)
-		(on_board yes)
-		(dnp no)
-		(fields_autoplaced yes)
-		(property "Reference" "J5"
-			(at 138.43 43.815 0)
-			(effects
-				(font
-					(size 1.27 1.27)
-				)
-			)
-		)
-		(property "Value" "Conn_01x03_Pin"
-			(at 135.89 43.815 0)
-			(effects
-				(font
-					(size 1.27 1.27)
-				)
-			)
-		)
-		(property "Footprint" ""
-			(at 130.81 43.18 0)
-			(effects
-				(font
-					(size 1.27 1.27)
-				)
-				(hide yes)
-			)
-		)
-		(property "Datasheet" "~"
-			(at 130.81 43.18 0)
-			(effects
-				(font
-					(size 1.27 1.27)
-				)
-				(hide yes)
-			)
-		)
-		(property "Description" "Generic connector, single row, 01x03, script generated"
-			(at 130.81 43.18 0)
-			(effects
-				(font
-					(size 1.27 1.27)
-				)
-				(hide yes)
-			)
-		)
-		(pin "3"
-		)
-		(pin "2"
-		)
-		(pin "1"
-		)
-		(instances
-			(project ""
-				(path "/fe75ec84-d622-42ca-b064-a5d970bee022"
-					(reference "J5")
-					(unit 1)
-				)
-			)
-		)
-	)
-	(symbol
 		(lib_id "Connector_Audio:AudioJack3_Ground")
 		(at 276.86 109.22 180)
@@
 					(unit 1)
 				)
+			)
+		)
+	)
+	(symbol
+		(lib_id "Connector:Conn_01x03_Pin")
+		(at 130.81 38.1 270)
+		(unit 1)
+		(exclude_from_sim no)
+		(in_bom yes)
+		(on_board yes)
+		(dnp no)
+		(fields_autoplaced yes)
+		(property "Reference" "J5"
+			(at 138.43 38.735 0)
+			(effects
+				(font
+					(size 1.27 1.27)
+				)
+			)
+		)
+		(property "Value" "Conn_01x03_Pin"
+			(at 135.89 38.735 0)
+			(effects
+				(font
+					(size 1.27 1.27)
+				)
+			)
+		)
+		(property "Footprint" "Connector_Hirose:Hirose_DF13-03P-1.25DSA_1x03_P1.25mm_Vertical"
+			(at 130.81 38.1 0)
+			(effects
+				(font
+					(size 1.27 1.27)
+				)
+				(hide yes)
+			)
+		)
+		(property "Datasheet" "~"
+			(at 130.81 38.1 0)
+			(effects
+				(font
+					(size 1.27 1.27)
+				)
+				(hide yes)
+			)
+		)
+		(property "Description" "Generic connector, single row, 01x03, script generated"
+			(at 130.81 38.1 0)
+			(effects
+				(font
+					(size 1.27 1.27)
+				)
+				(hide yes)
+			)
+		)
+		(pin "1"
+		)
+		(pin "2"
+		)
+		(pin "3"
+		)
+		(instances
+			(project "BrokeCW"
+				(path "/fe75ec84-d622-42ca-b064-a5d970bee022"
+					(reference "J5")
+					(unit 1)
+				)

Commit message: Add files via upload
Parts:
- removed R5, R7: R10K, Resistor_SMD:R_1210_3225Metric, symbol Device:R
- removed R8: R_Small, Resistor_SMD:R_0201_0603Metric, symbol Device:R_Small
- removed SW2, SW3, SW4, SW5, SW6: CK_KMS2xxGP, Button_Switch_SMD:SW_SPST_CK_KMS2xxGP, symbol Switch:CK_KMS2xxGP
- added R8: R, Resistor_SMD:R_0603_1608Metric, symbol Device:R
- added SW7: SW_Coded_SH-7050, Button_Switch_SMD:Nidec_Copal_SH-7010B, symbol Switch:SW_Coded_SH-7050
- C1, C2: footprint Capacitor_SMD:C_0805_2012Metric -> Capacitor_SMD:C_0603_1608Metric
- C3, C4: footprint Capacitor_THT:C_Disc_D5.1mm_W3.2mm_P5.00mm -> Capacitor_SMD:C_0603_1608Metric
- C5, C6: footprint Capacitor_THT:C_Disc_D7.0mm_W2.5mm_P5.00mm -> Capacitor_SMD:C_0805_2012Metric
- C7: footprint Capacitor_THT:C_Disc_D5.1mm_W3.2mm_P5.00mm -> Capacitor_SMD:C_0805_2012Metric
- C8, C9: footprint Capacitor_SMD:C_0402_1005Metric -> Capacitor_SMD:C_0805_2012Metric
- R1: footprint Resistor_SMD:R_2512_6332Metric -> Resistor_SMD:R_0805_2012Metric
- R2: footprint Resistor_SMD:R_1210_3225Metric -> Resistor_SMD:R_0603_1608Metric
- R3: footprint Resistor_SMD:R_1210_3225Metric -> Resistor_SMD:R_1206_3216Metric
- R4: footprint Resistor_SMD:R_2512_6332Metric -> Resistor_SMD:R_1206_3216Metric
- R6: footprint Resistor_THT:R_Axial_DIN0414_L11.9mm_D4.5mm_P15.24mm_Horizontal -> Resistor_SMD:R_1206_3216Metric
Connections:
- net at D3.2 (A): now also R8.1
- net at J7.10 (Pin_10): now also RV3.1, SW7.8
- net at J7.12 (Pin_12), J9.G, J9.T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: now also SW7.C
- net at J7.4 (Pin_4): now also SW7.1
- net at J7.8 (Pin_8): now also SW7.2
- net at J8.3 (Pin_3): now also R8.2

Commit message: Add files via upload
Parts:
- D1: footprint Diode_THT:D_DO-41_SOD81_P7.62mm_Horizontal -> Diode_SMD:D_SOD-323
- D2, D3: footprint LED_SMD:LED_0402_1005Metric -> LED_SMD:LED_0805_2012Metric
- Q1, Q2: footprint Package_TO_SOT_THT:TO-92_Inline -> Package_TO_SOT_SMD:SOT-23
Changed lines of the file:
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@@
 			)
 		)
-		(property "Footprint" "Package_TO_SOT_THT:TO-92_Inline"
+		(property "Footprint" "Package_TO_SOT_SMD:SOT-23"
 			(at 166.37 37.465 0)
 			(effects
@@
 			)
 		)
-		(property "Footprint" "LED_SMD:LED_0402_1005Metric"
+		(property "Footprint" "LED_SMD:LED_0805_2012Metric"
 			(at 133.35 147.32 0)
 			(effects
@@
 			)
 		)
-		(property "Footprint" "Package_TO_SOT_THT:TO-92_Inline"
+		(property "Footprint" "Package_TO_SOT_SMD:SOT-23"
 			(at 210.82 66.675 0)
 			(effects
@@
 			)
 		)
-		(property "Footprint" "Diode_THT:D_DO-41_SOD81_P7.62mm_Horizontal"
+		(property "Footprint" "Diode_SMD:D_SOD-323"
 			(at 120.65 64.77 90)
 			(effects
@@
 			)
 		)
-		(property "Footprint" "LED_SMD:LED_0402_1005Metric"
+		(property "Footprint" "LED_SMD:LED_0805_2012Metric"
 			(at 242.57 78.74 0)
 			(effects
