File: BrokeCW.kicad_pcb (KiCad board)
At the start: 2 copper layers, 222.2 x 71.8 mm, 44 parts, among them J1 Barrel_Jack_MountingPin, J10 AudioJack3_Radio, J2 Conn_Coaxial, J3 AudioJack3_Ground, J4 AudioJack3_Ground, J6 Conn_01x03_Pin, J7 Conn_01x15_PinLeft, J8 Conn_01x15_PinRight, J9 AudioJack3_Key, Q1 9013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

Commit message: Add files via upload
Parts:
- added J5: Conn_01x03_Pin, Connector_Hirose:Hirose_DF13-03P-1.25DSA_1x03_P1.25mm_Vertical, F.Cu at (157.5, 59.0)
- moved C7 0.50 mm to (216.5, 46.0)
- moved J6 0.25 mm to (157.5, 53.5)
Routing:
- net Net-(J5-Pin_1): track 50.2 -> 59.2 mm

Commit message: Add files via upload
Parts:
- removed R5, R7: R10K, Resistor_SMD:R_1210_3225Metric
- removed SW2, SW3, SW4, SW5, SW6: CK_KMS2xxGP, Button_Switch_SMD:SW_SPST_CK_KMS2xxGP
- added SW7: SW_Coded_SH-7050, Button_Switch_SMD:Nidec_Copal_SH-7010B, F.Cu at (63.5, 74.0)
- C1, C2: footprint Capacitor_SMD:C_0805_2012Metric -> Capacitor_SMD:C_0603_1608Metric
- C3, C4: footprint Capacitor_THT:C_Disc_D5.1mm_W3.2mm_P5.00mm -> Capacitor_SMD:C_0603_1608Metric
- C5, C6: footprint Capacitor_THT:C_Disc_D7.0mm_W2.5mm_P5.00mm -> Capacitor_SMD:C_0805_2012Metric
- C7: footprint Capacitor_THT:C_Disc_D5.1mm_W3.2mm_P5.00mm -> Capacitor_SMD:C_0805_2012Metric
- C8, C9: footprint Capacitor_SMD:C_0402_1005Metric -> Capacitor_SMD:C_0805_2012Metric
- R1: footprint Resistor_SMD:R_2512_6332Metric -> Resistor_SMD:R_0805_2012Metric
- R2: footprint Resistor_SMD:R_1210_3225Metric -> Resistor_SMD:R_0603_1608Metric
- R3: footprint Resistor_SMD:R_1210_3225Metric -> Resistor_SMD:R_1206_3216Metric
- R4: footprint Resistor_SMD:R_2512_6332Metric -> Resistor_SMD:R_1206_3216Metric
- R6: footprint Resistor_THT:R_Axial_DIN0414_L11.9mm_D4.5mm_P15.24mm_Horizontal -> Resistor_SMD:R_1206_3216Metric
- R8: value R_Small -> R; footprint Resistor_SMD:R_0201_0603Metric -> Resistor_SMD:R_0603_1608Metric
- moved C3 35.9 mm to (222.0, 79.8), turned to 90 degrees
- moved C8 20.1 mm to (207.4, 46.4)
- moved C9 20.1 mm to (216.9, 41.9)
- moved C1 20.1 mm to (211.9, 94.0)
- moved C4 20.1 mm to (220.4, 86.9)
- moved C7 20.1 mm to (196.4, 46.4)
- moved J2 20.1 mm to (227.5, 42.0)
- moved J3 20.1 mm to (233.3, 61.4)
- moved J4 20.1 mm to (234.1, 75.9)
- moved L2 20.1 mm to (216.0, 47.9)
- moved U1 20.1 mm to (202.2, 94.1)
- moved R1 9.98 mm to (171.5, 50.6)
- moved J9 9.28 mm to (50.8, 52.9)
- moved RV3 9.28 mm to (47.0, 69.5)
- moved R8 7.38 mm to (120.5, 56.5)
Connections:
- J7 pad 10: unconnected-(J7-Pin_10-Pad10) -> Net-(J7-Pin_10)
- J8 pad 6: Net-(J8-Pin_6) -> unconnected-(J8-Pin_6-Pad6)
- RV3 pad 1: unconnected-(RV3-Pad1) -> Net-(J7-Pin_10)
Routing:
- net Net-(J7-Pin_5): track 95.2 -> 0.00 mm
- net Net-(J7-Pin_12): track 147.0 -> 54.3 mm
- net Net-(J7-Pin_4): track 61.3 -> 0.00 mm
- net Net-(D1-A): track 290.7 -> 238.8 mm
- net Net-(J7-Pin_7): track 51.4 -> 0.00 mm
- net Net-(J8-Pin_6): track 43.6 -> 0.00 mm
- net Net-(D1-K): track 46.0 -> 10.3 mm
- net Net-(D2-K): track 235.8 -> 270.2 mm
- net Net-(C2-Pad1): track 26.8 -> 0.71 mm
- net Net-(J5-Pin_1): track 59.2 -> 33.6 mm
- net Net-(J7-Pin_10): track 0.00 -> 19.2 mm
- net Net-(Q1-C): track 42.3 -> 25.5 mm
- net Net-(J7-Pin_8): track 41.9 -> 25.9 mm
- net Net-(R6-Pad2): track 12.4 -> 26.1 mm
- net Net-(R7-Pad2): track 9.59 -> 0.00 mm
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Other:
- board size 222.2 x 71.8 mm -> 222.2 x 72.2 mm

Commit message: Add files via upload
Parts:
- D1: footprint Diode_THT:D_DO-41_SOD81_P7.62mm_Horizontal -> Diode_SMD:D_SOD-323
- D2, D3: footprint LED_SMD:LED_0402_1005Metric -> LED_SMD:LED_0805_2012Metric
- Q1, Q2: footprint Package_TO_SOT_THT:TO-92_Inline -> Package_TO_SOT_SMD:SOT-23
- moved C6 21.6 mm to (143.5, 63.0), turned to 180 degrees
- moved R2 17.0 mm to (177.8, 50.0), turned to 0 degrees
- moved L3 15.7 mm to (184.0, 67.5), turned to 0 degrees
- moved RV2 15.5 mm to (174.4, 79.1)
- moved C5 14.9 mm to (143.5, 58.5), turned to 180 degrees
- moved R6 14.2 mm to (184.5, 48.5), turned to 0 degrees
- moved C1 13.1 mm to (210.9, 81.0)
- moved C4 13.1 mm to (219.4, 73.9)
- moved U1 13.1 mm to (201.3, 81.1)
- moved C2 13.1 mm to (190.0, 84.0)
- moved C3 13.1 mm to (221.1, 66.8)
- moved L1 13.1 mm to (146.5, 82.0)
- moved R3 13.1 mm to (166.0, 86.0)
- moved D1 12.5 mm to (159.0, 45.0), turned to 90 degrees
- moved C7 9.91 mm to (190.1, 54.0)
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Routing:
- net Net-(J7-Pin_10): track 19.2 -> 85.1 mm
- net Net-(D2-A): track 155.0 -> 92.1 mm
- net Net-(D2-K): track 270.2 -> 224.5 mm
- net Net-(J7-Pin_5): track 0.00 -> 43.8 mm
- net Net-(J7-Pin_7): track 0.00 -> 42.9 mm
- net Net-(D1-A): track 238.8 -> 278.4 mm
- net Net-(J7-Pin_4): track 0.00 -> 34.9 mm
- net Net-(J7-Pin_12): track 54.3 -> 84.7 mm
- net Net-(Q2-C): track 51.7 -> 26.3 mm
- net Net-(D1-K): track 10.3 -> 32.9 mm
- net Net-(J5-Pin_1): track 33.6 -> 47.6 mm
- net Net-(J8-Pin_3): track 3.79 -> 17.0 mm
- net Net-(Q1-C): track 25.5 -> 37.4 mm
- net Net-(J7-Pin_8): track 25.9 -> 14.4 mm
- net Net-(R6-Pad2): track 26.1 -> 15.6 mm
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Other:
- board size 222.2 x 72.2 mm -> 197.2 x 59.2 mm
